File: LCDTemperatureHumidityMeter.sch (KiCad schematic (older format))
At the start: 11 parts, among them IC1 PIC16F1827, J1 Conn_02x01, M1 Octopus_DHT11, M2 SC1602, SW1 SW_Push

Commit message: 基板設計完了と，それに伴い配線の変更。
Connections:
- net GND: now also RV1.1, SW1.2; no longer RV1.3, SW1.1
- net VCC: now also RV1.3; no longer RV1.1
- net at M2.10 (D3): now also IC1.12 (RB6/ICSPCLK); no longer IC1.7 (RB1)
- net at M2.11 (D4): now also IC1.9 (RB3); no longer IC1.11 (RB5)
- net at M2.13 (D6): now also IC1.7 (RB1); no longer IC1.10 (RB4)
- net at M2.14 (D7): now also IC1.6 (RB0); no longer IC1.9 (RB3)
- net at M2.4 (RS): now also IC1.17 (RA0); no longer IC1.18 (RA1)
- net at M2.5 (R/W): now also IC1.15 (RA6); no longer IC1.17 (RA0)
- net at M2.7 (D0): now also IC1.11 (RB5); no longer IC1.13 (RB7/ICSPDAT)
- net at M2.8 (D1): now also IC1.10 (RB4); no longer IC1.6 (RB0)
- net at M2.9 (D2): now also IC1.13 (RB7/ICSPDAT); no longer IC1.12 (RB6/ICSPCLK)
- net at IC1.1 (RA2): no longer M1.3 (Signal)
- net at IC1.3 (RA4): now also M1.3 (Signal)
- net at IC1.4 (RA5/MCLR), R1.2: now also SW1.1; no longer SW1.2
Changed lines of the file:
@@
 	2100 2300 2000 2300
 Wire Wire Line
-	2000 2300 2000 3450
-Wire Wire Line
-	1900 2200 1900 3250
-Wire Wire Line
 	1900 2200 2100 2200
 Wire Wire Line
 	2100 2100 1800 2100
-Wire Wire Line
-	1800 2100 1800 3050
-Wire Wire Line
-	1700 2000 1700 2850
 Wire Wire Line
 	1700 2000 2100 2000
@@
 F 3 "" H 5350 2250 50  0001 C CNN
 	1    5350 2250
-	-1   0    0    -1
+	-1   0    0    1
 $EndComp
 Wire Wire Line
@@
 F 3 "" H 1350 2300 50  0001 C CNN
 	1    1350 2100
-	0    -1   -1   0
+	0    -1   1    0
 $EndComp
 Wire Wire Line
@@
 $EndComp
 Wire Wire Line
-	2100 1500 1550 1500
-Wire Wire Line
-	1550 1500 1550 1350
-Wire Wire Line
-	3100 1500 3600 1500
-Wire Wire Line
-	3600 1500 3600 2450
-Wire Wire Line
-	3100 1600 3700 1600
-Wire Wire Line
-	3700 1600 3700 2350
-Wire Wire Line
-	3100 1700 3800 1700
-Wire Wire Line
-	3800 1700 3800 2250
+	1550 1350 1550 1700
 Wire Wire Line
 	3100 2000 3500 2000
@@
 Wire Wire Line
 	3200 2300 3100 2300
-Wire Wire Line
-	2000 3450 3900 3450
-Wire Wire Line
-	1900 3250 3900 3250
-Wire Wire Line
-	1800 3050 3900 3050
-Wire Wire Line
-	1700 2850 3900 2850
-Wire Wire Line
-	3200 2300 3200 3350
-Wire Wire Line
-	3200 3350 3900 3350
-Wire Wire Line
-	3300 2200 3300 3150
-Wire Wire Line
-	3300 3150 3900 3150
-Wire Wire Line
-	3400 2950 3900 2950
-Wire Wire Line
-	3400 2950 3400 2100
-Wire Wire Line
-	3500 2000 3500 2750
-Wire Wire Line
-	3500 2750 3900 2750
 $Comp
 L Conn_02x01 J1
@@
 	0    1    1    0
 $EndComp
+Wire Wire Line
+	1700 2000 1700 3450
+Wire Wire Line
+	1700 3450 3900 3450
+Wire Wire Line
+	1800 2100 1800 3350
+Wire Wire Line
+	1800 3350 3900 3350
+Wire Wire Line
+	1900 3250 3900 3250
+Wire Wire Line
+	1900 3250 1900 2200
+Wire Wire Line
+	2000 2300 2000 3150
+Wire Wire Line
+	2000 3150 3900 3150
+Wire Wire Line
+	3500 2000 3500 2950
+Wire Wire Line
+	3500 2950 3900 2950
+Wire Wire Line
+	3400 2100 3400 3050
+Wire Wire Line
+	3400 3050 3900 3050
+Wire Wire Line
+	3300 2200 3300 2750
+Wire Wire Line
+	3300 2750 3900 2750
+Wire Wire Line
+	3200 2300 3200 2850
+Wire Wire Line
+	3200 2850 3900 2850
+Wire Wire Line
+	3100 1800 3700 1800
+Wire Wire Line
+	3700 1800 3700 2350
+Wire Wire Line
+	3100 1700 3800 1700
+Wire Wire Line
+	3800 1700 3800 2250
+Wire Wire Line
+	3600 2450 3600 1600
+Wire Wire Line
+	3600 1600 3100 1600
+Wire Wire Line
+	1550 1700 2100 1700
 $EndSCHEMATC
